File: esquematicos/tp_final_circuito/tp_final_circuito.kicad_sch (KiCad schematic)
At the start: 21 parts, among them SW1 SW_DIP_x08, SW2 BOTON CONFIG, SW3 BOTON ENTER, SW4 BOTON NEXT, SW5 BOTON ESC, SW6 BOTON INGRESO, SW7 BOTON EGRESO, U1 NUCLEO-F410RB, U2 LM35-LP, U3 Buzzer

Commit message: Uso de cpu y mejora de interfaz
Other:
- company: (none) -> FIUBA
- title: (none) -> TdSE: TP Final Puerta Esclusa
Changed lines of the file:
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@@
 (kicad_sch (version 20230121) (generator eeschema)
   (paper "A4")
+  (title_block
+    (title "TdSE: TP Final Puerta Esclusa")
+    (date "2024-12-11")
+    (company "FIUBA")
+  )
   (junction (at 255.27 69.85) (diameter 0) (color 0 0 0 0)
   )
